File: Hardware/OpenBook.brd (EAGLE design)
At the start: 170.2 x 111.2 mm, 103 parts, among them IC1 BD5229G-TR, IC4 XC6220A331MR-G, J1 FH34SRJ-24S-0.5SH_99_, J10 112A-TAAR-R03_ATTEND, J2 SAMACSYS_PARTS_USB4110-GF-A, J3 QWIIC_RIGHT_ANGLE, Q1 20V/4.2A/52mΩ/1.4W, Q2 20V/4.2A/52mΩ/1.4W, Q3 SI1308EDL-T1-GE3, U1 W25Q512JVEIQ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

Commit message: Add 3D model
Parts:
- moved J2 0.85 mm to (167.8, 54.5)
- moved C6 0.74 mm to (27.2, 108.8)
- moved C5 0.61 mm to (52.5, 108.8)
- moved C10 0.58 mm to (67.1, 108.8)
- moved BOOT_BUTTON 0.43 mm to (23.9, 108.9)
- moved RESET_BUTTON 0.38 mm to (49.1, 108.9)
- moved J3 0.27 mm to (165.5, 19.5)
- moved IC1 0.24 mm to (49.2, 102.8)
- moved C_DELAY 0.24 mm to (52.4, 102.9)
- moved R_RESET 0.23 mm to (45.6, 108.6)
- moved R_BOOT 0.23 mm to (20.7, 108.7)
- moved CHANGE_BUTTON 0.20 mm to (63.8, 108.9)
- moved R_CHANGE 0.19 mm to (60.5, 108.7)
Routing:
- net EPD_RST: track 140.1 -> 110.5 mm
- net RESE: track 56.2 -> 32.6 mm
- net MOSI: track 193.5 -> 174.3 mm
- net EPD_DC: track 106.5 -> 115.9 mm
- net FLASH_CS: track 27.7 -> 37.1 mm, vias 4 -> 2
- net SS_SD: track 76.8 -> 68.4 mm
- net INT_RTC: track 81.1 -> 85.9 mm, vias 4 -> 5
- net EPD_BUSY: track 121.8 -> 126.5 mm
- net GND: track 789.1 -> 784.7 mm
- net SCK: track 189.4 -> 191.7 mm, vias 8 -> 7
- net 3V3: track 424.0 -> 426.1 mm
- net USB_D+: track 147.9 -> 145.9 mm
- net SCL: track 205.9 -> 207.7 mm
- net IO/BOOT: track 55.2 -> 53.5 mm
- net USB_D-: track 149.8 -> 148.0 mm
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- added copper zone on layer 1, net GND
- added copper zone on layer 16, net GND
Other:
- board text added: "L1"
- board text added: "U2"
- board text removed: "ESP32"
