File: Hardware/OpenBook.sch (EAGLE design)
At the start: 103 parts, among them IC1 BD5229G-TR, IC4 XC6220A331MR-G, J1 FH34SRJ-24S-0.5SH_99_, J10 112A-TAAR-R03_ATTEND, J2 SAMACSYS_PARTS_USB4110-GF-A, J3 QWIIC_RIGHT_ANGLE, Q1 20V/4.2A/52mΩ/1.4W, Q2 20V/4.2A/52mΩ/1.4W, Q3 SI1308EDL-T1-GE3, U1 W25Q512JVEIQ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

Commit message: Update sch
Other:
- note added: "Drawn by: Radu Marin"
- note removed: "Drawn by Radu Marin"
- moved on the sheet: BOOT_BUTTON, C1, C10, C10_SUPERCAP, C1_BAT, C1_BAT1, C1_BAT2, C2, C2_BAT, C3, C4, C4_USB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

Commit message: Update sch
Parts:
- CHG_LED: value (none) -> SMD-LED0603
- SJ1: value (none) -> 1m
Other:
- note added: "21/03/2025 20:24PM"
- note added: "DeskAssistant"
- note added: "Drawn by Radu Marin"
- note removed: "21/03/2025 20:24 PM"
- note removed: "DeskAssistant v19"
- note removed: "Drawn by: Radu Marin"
- moved on the sheet: BOOT_BUTTON, C1, C10, C10_SUPERCAP, C1_BAT, C1_BAT1, C1_BAT2, C2, C2_BAT, C3, C4, C4_USB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
